Commit message: Update robot.urdf

File: Gazebo/robot.urdf (robot description, URDF)
Before this commit: robot box_bot, 5 links, 4 joints
Links:
- removed link back_left_wheel
- removed link back_right_wheel
- added link rear_left_wheel, mass 0.5; collision cylinder length=0.05 radius=0.10; visual cylinder length=0.05 radius=0.10
- added link rear_right_wheel, mass 0.5; collision cylinder length=0.05 radius=0.10; visual cylinder length=0.05 radius=0.10
- link base_link: mass 5.0 -> 10.0; geometry collision box size=0.60 0.40 0.20; visual box size=0.60 0.40 0.20
- link front_left_wheel: geometry collision cylinder length=0.05 radius=0.10; visual cylinder length=0.05 radius=0.10
- link front_right_wheel: geometry collision cylinder length=0.05 radius=0.10; visual cylinder length=0.05 radius=0.10
Joints:
- removed joint back_left_wheel_joint
- removed joint back_right_wheel_joint
- added joint rear_left_wheel_joint: type continuous, parent base_link, child rear_left_wheel, origin xyz=-0.20 0.225 0 rpy=0 0 0, axis 0 1 0
- added joint rear_right_wheel_joint: type continuous, parent base_link, child rear_right_wheel, origin xyz=-0.20 -0.225 0 rpy=0 0 0, axis 0 1 0
- joint front_left_wheel_joint: origin xyz=0.2 0.25 -0.1 rpy=-1.5707 0 0 -> xyz=0.20 0.225 0 rpy=0 0 0
- joint front_right_wheel_joint: origin xyz=0.2 -0.25 -0.1 rpy=-1.5707 0 0 -> xyz=0.20 -0.225 0 rpy=0 0 0

Commit message: Add lidar sensor and base footprint to robot model
Added lidar sensor and updated robot structure with base footprint.

File: Gazebo/robot.urdf (robot description, URDF)
Before this commit: robot box_bot, 5 links, 4 joints
Links:
- added link base_footprint
- added link lidar_link, mass 0.1; collision cylinder length=0.1 radius=0.05; visual cylinder length=0.1 radius=0.05
Joints:
- added joint base_footprint_joint: type fixed, parent base_footprint, child base_link, origin xyz=0 0 0.1 rpy=0 0 0
- added joint lidar_joint: type fixed, parent base_link, child lidar_link, origin xyz=0 0 0.15 rpy=0 0 0

Commit message: Add files via upload

File: Gazebo/robot.urdf (robot description, URDF)
Before this commit: robot box_bot, 7 links, 6 joints
Links:
- added link camera_link, mass 0.05; collision box size=0.05 0.05 0.05; visual box size=0.05 0.05 0.05
Joints:
- added joint camera_joint: type fixed, parent base_link, child camera_link, origin xyz=0.3 0 0.1 rpy=0 0 0

Commit message: Add files via upload
Updated Sim + fixed bugs. Lidar now only 180 degrees, can be changed in robot.urdf

File: Gazebo/robot.urdf (robot description, URDF)
Before this commit: robot box_bot, 8 links, 7 joints
Links:
- added link imu_link, mass 0.01; collision box size=0.02 0.02 0.02; visual box size=0.02 0.02 0.02
Joints:
- added joint imu_joint: type fixed, parent base_link, child imu_link, origin xyz=0 0 0.1 rpy=0 0 0
